Commit message: fix xyz to zyx bug

File: urdf/mano.urdf (robot description, URDF)
Before this commit: robot mano, 23 links, 22 joints
Links:
- link thumb1x: geometry 
- link thumb1z: geometry collision mesh filename=urdf_meshes/thumb1_collision.obj; visual mesh filename=urdf_meshes/thumb1_vis.obj
Joints:
- joint j_thumb1x: origin xyz=0.0 0.0 0.0 rpy=0.0 -0.0 0.0 -> xyz=-0.02408969 -0.01552234  0.02581285 rpy=1.3934614224320991 0.7332206451663358 0.5723973954752037; parent thumb1y -> palm
- joint j_thumb1y: origin xyz=0.0, 0.0, 0.0 rpy=0.0 -0.0 0.0 -> xyz=0.0 0.0 0.0 rpy=0.0 -0.0 0.0; parent thumb1z -> thumb1x
- joint j_thumb1z: origin xyz=-0.02408969 -0.01552234  0.02581285 rpy=1.3934614224320991 0.7332206451663358 0.5723973954752037 -> xyz=0.0 0.0 0.0 rpy=0.0 -0.0 0.0; parent palm -> thumb1y
- joint j_thumb2y: parent thumb1x -> thumb1z
- joint j_thumb2z: origin xyz=0.0, 0.0, 0.0 rpy=0.0 -0.0 0.0 -> xyz=0.0 0.0 0.0 rpy=0.0 -0.0 0.0
